File: KiCAD/Amiga-Rejuvenator/Amiga-Rejuvenator.sch (KiCad schematic (older format))
At the start: 120 parts, among them J1 GND, J15 28M, J17 RMBCLKS, J18 GND, J19 +12X, U1 74LS245, U10 V53C104, U11 V53C104, U12 V53C104, U13 V53C104, U14 74LS244-U16,U17, U15 74LS373, U16 74LS244-U16,U17, U17 74LS244-U16,U17, U18 512K-ROM, U19 8372-FatAgnus, U19B1 8361-Agnus, U2 74LS393-U2, U20 8364-Paula, U20B1 8364-Paula, U21 74LS245, U22 74LS245, U23 RP, U24 RP, U25 8362-Denise, U25B1 8362-Denise, U26 74HC245, U27 OKI6242B, U28 PAL16L8, U29 PAL16L8, U3 74F257, U30 PAL20L8, U31 PAL20L8, U32 74LS74, U33 74LS04, U34 74HC245, U35 74F257, U36 PALCAS, U37 PALEN, U38 U3I, U39 U3G, U4 74LS244-U16,U17, U40 U2J, U41 U2I, U5 74LS373, U6 V53C104, U7 V53C104, U8 V53C104, U9 V53C104, X1 X1, X14 X14, X15 X15, X16 VideoSlot 1, X17 VideoSlot 2, Y1 Crystal

Commit message: Signal name updates
Signal name updates on KiCAD schematics and board artwork.
Connections:
- net ~ARW: now reaches U36.1
- net REJ.1 renamed REJ1
- net REJ.2 renamed REJ2
- net REJ.3 renamed REJ3
- net REJ.4 renamed ~CNT
- net REJ.KICK renamed REJKICK
- net REJ.MCFG1 renamed MCFG1
- net REJ.MCFG2 renamed MCFG2
- net REJ.~CE renamed ~DAE
- net REJ.~OE1 renamed ~CDRREJ
- net REJ.~OE2 renamed ~CDWREJ
- net RTC.~RD renamed ~CLKR
- net RTC.~WR renamed ~CLKW
- net RW renamed ~PRW
- net ~MYRAME renamed ~ROME
Other:
- note removed: "? ~WPRO"
- note removed: "_CDR"
- note removed: "_CDW"
- note removed: "_CNT"
- note removed: "~ARW"
Changed lines of the file:
@@
 $EndComp
 $Comp
+L Logic_Programmable:PAL20L8 U30
+U 1 1 5B83B3CF
+P 14850 10900
+F 0 "U30" H 14550 11700 50  0000 C CNN
+F 1 "PAL20L8" H 15050 11700 50  0000 C CNN
+F 2 "Package_DIP:DIP-24_W7.62mm" H 14850 10900 50  0001 C CNN
+F 3 "" H 14850 10900 50  0001 C CNN
+	1    14850 10900
+	1    0    0    -1
+$EndComp
+$Comp
 L Amiga-Rejuvenator:OKI6242B U27
 U 1 1 5B83D629
@@
 ~RESET
 Text Label 22450 7650 0    50   ~ 0
-REJ.KICK
+REJKICK
 Text Label 15400 13200 0    50   ~ 0
-REJ.KICK
+REJKICK
 Text Label 14300 7500 2    50   ~ 0
-REJ.1
+REJ1
 Text Label 15400 10600 0    50   ~ 0
-REJ.1
+REJ1
 $Comp
 L power:+5V #PWR0170
@@
 	13150 11400 14350 11400
 Text Label 14300 11400 2    50   ~ 0
-RW
+~PRW
 Entry Wire Line
 	22250 6800 22150 6700
@@
 	23000 6800 22250 6800
 Text Label 22750 6800 2    50   ~ 0
-RW
+~PRW
 Wire Wire Line
 	13150 11500 14350 11500
@@
 ~RE
 Text Label 14300 10400 2    50   ~ 0
-REJ.2
+REJ2
 Text Label 15400 13800 0    50   ~ 0
-REJ.2
+REJ2
 $Comp
 L 74xx:74LS245 U1
@@
 $EndComp
 Text Label 5550 3750 2    50   ~ 0
-REJ.~CE
+~DAE
 Wire Wire Line
 	13150 10500 14350 10500
 Text Label 14300 10500 2    50   ~ 0
-REJ.~CE
+~DAE
 Text Label 15400 13300 0    50   ~ 0
-REJ.~CE
+~DAE
 Wire Wire Line
 	13150 10800 14350 10800
@@
 ~C3
 Text Label 15400 7100 0    50   ~ 0
-REJ.3
+REJ3
 Text Label 14300 13100 2    50   ~ 0
-REJ.MCFG2
+MCFG2
 $Comp
 L Device:R_Network09_US RP5
@@
 $EndComp
 Text Label 12450 13100 0    50   ~ 0
-REJ.MCFG2
+MCFG2
 $Comp
 L Device:Jumper_NC_Small JP101
@@
 $EndComp
 Text Label 12450 13000 0    50   ~ 0
-REJ.MCFG1
+MCFG1
 Text Label 14300 14400 2    50   ~ 0
-REJ.MCFG1
+MCFG1
 Text Label 14300 13600 2    50   ~ 0
 A20
@@
 ~BLS
 Text Label 15400 7700 0    50   ~ 0
-~MYRAME
+~ROME
 Text Label 15400 7800 0    50   ~ 0
 ~VPA
@@
 ~REGEN
 Text Label 9000 6150 0    50   ~ 0
-RTC.~RD
+~CLKR
 Text Label 15400 10900 0    50   ~ 0
-RTC.~RD
+~CLKR
 $Comp
 L Amiga-Rejuvenator:74LS393-U2 U2
@@
 $EndComp
 Text Label 15400 10800 0    50   ~ 0
-REJ.~OE1
+~CDRREJ
 Entry Wire Line
 	10550 12250 10450 12350
 Text Label 9750 12350 2    50   ~ 0
-REJ.~OE1
+~CDRREJ
 Entry Wire Line
 	10550 10450 10450 10550
@@
 	10450 10550 9450 10550
 Text Label 9750 10550 2    50   ~ 0
-REJ.~OE1
+~CDRREJ
 Text Label 15400 10700 0    50   ~ 0
-REJ.~OE2
+~CDWREJ
 Entry Wire Line
 	10550 13950 10450 14050
@@
 	10450 14050 9500 14050
 Text Label 9850 14050 2    50   ~ 0
-REJ.~OE2
+~CDWREJ
 Entry Wire Line
 	10550 8450 10450 8550
@@
 	10450 8550 9500 8550
 Text Label 9850 8550 2    50   ~ 0
-REJ.~OE2
+~CDWREJ
 Wire Wire Line
 	12100 13200 12200 13200
 Text Label 12450 12550 0    50   ~ 0
-REJ.KICK
+REJKICK
 NoConn ~ 12100 13300
 NoConn ~ 12100 13400
@@
 NoConn ~ 12100 13800
 Text Label 15400 10500 0    50   ~ 0
-REJ.4
+~CNT
 Text Label 5700 1200 2    50   ~ 0
-REJ.4
+~CNT
 NoConn ~ 15350 10400
 NoConn ~ 15350 10300
 Text Label 9000 5950 0    50   ~ 0
-RTC.~WR
+~CLKW
 Text Label 15400 10200 0    50   ~ 0
-RTC.~WR
+~CLKW
 Wire Wire Line
 	7800 8550 7500 8550
@@
 Text Notes 6850 11250 0    50   ~ 0
 MB\n74LS244
-$Comp
-L Amiga-Rejuvenator:Board2Board[20-pin] U36
-U 1 1 5ECAE079
-P 14850 2700
-F 0 "U36" H 14600 3300 50  0000 C CNN
-F 1 "PALCAS" H 14850 2750 79  0000 C CNN
-F 2 "MOLEX_4455:MOLEX_4455-10_W7.62mm[x2-R]" H 14850 2750 50  0001 C CNN
-F 3 "~" H 14850 2750 50  0001 C CNN
-	1    14850 2700
-	1    0    0    -1
-$EndComp
 Wire Wire Line
 	15500 3100 15300 3100
@@
 A19
 Text Label 14350 2500 2    50   ~ 0
-RW
+~PRW
 Text Label 14350 2600 2    50   ~ 0
 ~UDS
@@
 	0    1    1    0
 $EndComp
-Text Notes 14200 2200 0    50   ~ 0
-~ARW
 Text Notes 14350 2800 2    50   ~ 0
 ~ROME
@@
 ~DTACK
 Text Label 15300 6400 0    50   ~ 0
-~MYRAME
+~ROME
 Text Label 15300 6500 0    50   ~ 0
 ~VPA
@@
 NoConn ~ 15400 4200
 Text Label 14350 3600 2    50   ~ 0
-REJ.3
+REJ3
 Text Label 14350 4500 2    50   ~ 0
 ~AS
@@
 A18
 Text Label 14350 3900 2    50   ~ 0
-RW
+~PRW
 Wire Wire Line
 	13150 3900 14400 3900
 Text Label 14350 4200 2    50   ~ 0
-REJ.KICK
+REJKICK
 Wire Wire Line
 	13150 4200 14400 4200
@@
 C4
 Text Label 10400 3250 2    50   ~ 0
-REJ.~CE
+~DAE
 Text Label 10400 3050 2    50   ~ 0
-REJ.4
+~CNT
 Wire Wire Line
 	3500 7850 4300 7850
@@
 Text Notes 15700 13800 0    50   ~ 0
 _CLKE
-Text Notes 15700 13300 0    50   ~ 0
-_DAE
 Text Notes 13850 10400 0    50   ~ 0
 _CLKE
 Text Notes 13650 10500 0    50   ~ 0
 _DAE
-Text Notes 15750 10700 0    50   ~ 0
-_CDW
-Text Notes 15750 10800 0    50   ~ 0
-_CDR
-Text Notes 15700 10500 0    50   ~ 0
-_CNT
-Text Notes 9900 3050 0    50   ~ 0
-_CNT
-Text Notes 9900 3250 0    50   ~ 0
-_DAE
 Connection ~ 11800 14350
 Wire Wire Line
@@
 	12300 13000 12950 13000
 $Comp
-L Logic_Programmable:PAL20L8 U30
-U 1 1 5B83B3CF
-P 14850 10900
-F 0 "U30" H 14550 11700 50  0000 C CNN
-F 1 "PAL20L8" H 15050 11700 50  0000 C CNN
-F 2 "Package_DIP:DIP-24_W7.62mm" H 14850 10900 50  0001 C CNN
-F 3 "" H 14850 10900 50  0001 C CNN
-	1    14850 10900
+L Amiga-Rejuvenator:Board2Board[20-pin] U36
+U 1 1 5ECAE079
+P 14850 2700
+F 0 "U36" H 14600 3300 50  0000 C CNN
+F 1 "PALCAS" H 14850 2750 79  0000 C CNN
+F 2 "MOLEX_4455:MOLEX_4455-10_W7.62mm[x2-R]" H 14850 2100 50  0001 C CNN
+F 3 "~" H 14850 2100 50  0001 C CNN
+	1    14850 2700
 	1    0    0    -1
 $EndComp
-Text Notes 15450 4200 0    50   ~ 0
-? ~WPRO
+Text Label 14200 2200 0    50   ~ 0
+~ARW
 Wire Wire Line
 	12400 13100 14350 13100

Commit message: Signal names and active low status updated
Connections:
- net REJ1 renamed _REJ1
- net REJ2 renamed _REJ2
- net REJ3 renamed _REJ3
Other:
- note removed: "_DAE"
Changed lines of the file:
@@
 REJKICK
 Text Label 14300 7500 2    50   ~ 0
-REJ1
+_REJ1
 Text Label 15400 10600 0    50   ~ 0
-REJ1
+_REJ1
 $Comp
 L power:+5V #PWR0170
@@
 ~RE
 Text Label 14300 10400 2    50   ~ 0
-REJ2
+_REJ2
 Text Label 15400 13800 0    50   ~ 0
-REJ2
+_REJ2
 $Comp
 L 74xx:74LS245 U1
@@
 ~C3
 Text Label 15400 7100 0    50   ~ 0
-REJ3
+_REJ3
 Text Label 14300 13100 2    50   ~ 0
 MCFG2
@@
 ~ROM01
 NoConn ~ 15400 4200
-Text Label 14350 3600 2    50   ~ 0
-REJ3
 Text Label 14350 4500 2    50   ~ 0
 ~AS
@@
 Text Notes 15700 13800 0    50   ~ 0
 _CLKE
-Text Notes 13850 10400 0    50   ~ 0
+Text Notes 13800 10400 0    50   ~ 0
 _CLKE
-Text Notes 13650 10500 0    50   ~ 0
-_DAE
 Connection ~ 11800 14350
 Wire Wire Line
@@
 Text Label 14200 2200 0    50   ~ 0
 ~ARW
+Text Label 14350 3600 2    50   ~ 0
+_REJ3
 Wire Wire Line
 	12400 13100 14350 13100

Commit message: Add directional signals for Agnus.  Add PWR_FLAG for power inputs.
Connections:
- net +BATT: now reaches BT1.1 (+), BT1.2 (+), C30.1, R3.2
Changed lines of the file:
@@
 Wire Wire Line
 	7450 3800 7450 3750
-Wire Wire Line
-	7450 3750 7900 3750
 Connection ~ 7450 3750
 Wire Wire Line
@@
 	7400 4200 7400 4250
 Wire Wire Line
-	7400 4250 7200 4250
+	7400 4250 7300 4250
 $Comp
 L Amiga-Rejuvenator:3.6V_Varta BT1
@@
 	7500 4250 7550 4250
 Wire Wire Line
-	7500 4250 7400 4250
+	7500 4250 7450 4250
 Connection ~ 7500 4250
 Connection ~ 7400 4250
@@
 	0    1    -1   0
 $EndComp
-Text Label 8250 4250 2    50   ~ 0
-BATT+
 $Comp
 L Amiga-Rejuvenator:V53C104 U10
@@
 Connection ~ 10150 4100
 Wire Wire Line
-	10150 4200 10150 4950
+	10150 4200 10150 4500
 Connection ~ 10150 4200
 Connection ~ 10150 4950
@@
 	10250 4400 10100 4400
 Wire Wire Line
-	10250 4400 10250 4750
+	10250 4400 10250 4500
 Connection ~ 10250 4400
 Connection ~ 10250 4750
@@
 Text Label 14350 3600 2    50   ~ 0
 _REJ3
+$Comp
+L power:PWR_FLAG #FLG0101
+U 1 1 6124A46E
+P 10150 4500
+F 0 "#FLG0101" H 10150 4575 50  0001 C CNN
+F 1 "PWR_FLAG" V 10150 4627 50  0000 L CNN
+F 2 "" H 10150 4500 50  0001 C CNN
+F 3 "~" H 10150 4500 50  0001 C CNN
+	1    10150 4500
+	0    -1   -1   0
+$EndComp
+Connection ~ 10150 4500
+Wire Wire Line
+	10150 4500 10150 4950
+$Comp
+L power:PWR_FLAG #FLG0102
+U 1 1 6124EFBD
+P 10250 4500
+F 0 "#FLG0102" H 10250 4575 50  0001 C CNN
+F 1 "PWR_FLAG" H 10050 4650 50  0000 L CNN
+F 2 "" H 10250 4500 50  0001 C CNN
+F 3 "~" H 10250 4500 50  0001 C CNN
+	1    10250 4500
+	0    1    1    0
+$EndComp
+Connection ~ 10250 4500
+Wire Wire Line
+	10250 4500 10250 4750
+$Comp
+L power:PWR_FLAG #FLG0103
+U 1 1 61252952
+P 7700 5000
+F 0 "#FLG0103" H 7700 5075 50  0001 C CNN
+F 1 "PWR_FLAG" H 7700 5173 50  0000 C CNN
+F 2 "" H 7700 5000 50  0001 C CNN
+F 3 "~" H 7700 5000 50  0001 C CNN
+	1    7700 5000
+	-1   0    0    1
+$EndComp
+Connection ~ 7700 5000
+$Comp
+L power:PWR_FLAG #FLG0104
+U 1 1 61256223
+P 7450 4250
+F 0 "#FLG0104" H 7450 4325 50  0001 C CNN
+F 1 "PWR_FLAG" H 7200 4350 50  0000 C CNN
+F 2 "" H 7450 4250 50  0001 C CNN
+F 3 "~" H 7450 4250 50  0001 C CNN
+	1    7450 4250
+	-1   0    0    1
+$EndComp
+Connection ~ 7450 4250
+Wire Wire Line
+	7450 4250 7400 4250
+Text Label 8250 4250 2    50   ~ 0
+BATT+
+$Comp
+L power:+BATT #PWR0129
+U 1 1 612661B9
+P 7300 4250
+F 0 "#PWR0129" H 7300 4100 50  0001 C CNN
+F 1 "+BATT" H 7300 4200 50  0000 C CNN
+F 2 "" H 7300 4250 50  0001 C CNN
+F 3 "" H 7300 4250 50  0001 C CNN
+	1    7300 4250
+	1    0    0    -1
+$EndComp
+Connection ~ 7300 4250
+Wire Wire Line
+	7300 4250 7200 4250
+Wire Wire Line
+	7450 3750 7900 3750
 Wire Wire Line
 	12400 13100 14350 13100

Commit message: Signaling Update
Updated signal direction for RAM, custom chips, and motherboard headers.  Rejuvenator now completes the ERC check error free!  (It previously had errors due to missing signal directions on the symbol entries.)

Renamed nets that are connected by way of the mainboard.  Previously, these nets were named (for example) X2.~CDW, X9.~CDW, X15.~CDW.  Now these same signals would be named ~CDWa, ~CDWb, ~CDWc.   Keep in mind, these are all the same signal.  They are not connected on the rejuvenator itself, but they become interconnected once plugged to the mainboard.  For example, all the CDWa,b,c signals are the same CDW signal, just fed up to Rejuvenator from different points on the mainboard.
Parts:
- removed U19B1: 8361-Agnus, Package_DIP:DIP-48_W15.24mm_Socket, symbol Amiga-Rejuvenator:8361-Agnus
- removed U20B1: 8364-Paula, MOLEX_4455:48pin_blank_socket, symbol Amiga-Rejuvenator:8364-Paula
- removed U25B1: 8362-Denise, MOLEX_4455:48pin_blank_socket, symbol Amiga-Rejuvenator:8362-Denise
- added U19B1: 8361-Agnus-Socket, Package_DIP:DIP-48_W15.24mm_Socket, symbol Amiga-Rejuvenator:8361-Agnus-Socket
- added U20B1: 8364-Paula-Socket, MOLEX_4455:48pin_blank_socket, symbol Amiga-Rejuvenator:8364-Paula-Socket
- added U25B1: 8362-Denise-Socket, MOLEX_4455:48pin_blank_socket, symbol Amiga-Rejuvenator:8362-Denise-Socket
Connections:
- net +5V: now also U19B1.10 (Vcc), U20B1.27 (Vcc), U25B1.19 (Vcc)
- net 7M: now also U25B1.35 (7M)
- net ANAGND: now also U20B1.34 (ANAGND)
- net AUDL: now also U20B1.31 (AUDL)
- net AUDR: now also U20B1.30 (AUDR)
- net B0: now also U25B1.24 (B0)
- net B1: now also U25B1.25 (B1)
- net B2: now also U25B1.26 (B2)
- net B3: now also U25B1.27 (B3)
- net CCK.OA: now also U19B1.25 (CCK)
- net CCK.P: now also U20B1.28 (CCK)
- net CCKQ.OA: now also U19B1.26 (CCKQ)
- net CCKQ.P: now also U20B1.29 (CCKQ)
- net DMAL: now also U20B1.12 (DMAL)
- net G0: now also U25B1.28 (G0)
- net G1: now also U25B1.29 (G1)
- net G2: now also U25B1.30 (G2)
- net G3: now also U25B1.31 (G3)
- net GND: now also U19B1.27 (GND), U20B1.8 (GND), U25B1.37 (GND)
- net M0H: now also U25B1.9 (M0H)
- net M0V: now also U25B1.38 (M0V)
- net M1H: now also U25B1.8 (M1H)
- net M1V: now also U25B1.39 (M1V)
- net POT0X: now also U20B1.32 (POT0X)
- net POT0Y: now also U20B1.33 (POT0Y)
- net POT1X: now also U20B1.35 (POT1X)
- net POT1Y: now also U20B1.36 (POT1Y)
- net R0: now also U25B1.20 (R0)
- net R1: now also U25B1.21 (R1)
- net R2: now also U25B1.22 (R2)
- net R3: now also U25B1.23 (R3)
- net RxD: now also U20B1.41 (RxD)
- net TxD: now also U20B1.40 (TxD)
- net ~BURST: now also U25B1.18 (~BURST)
- net ~CAS: now also U25B1.36 (~CAS)
- net ~CSYNC: now also U19B1.39 (~CSYNC)
- net ~DKRD: now also U20B1.37 (~DKRD)
- net ~DKWD: now also U20B1.38 (~DKWD)
- net ~DKWE: now also U20B1.39 (DKWE)
- net ~HSYNC: now also U19B1.40 (~HSYNC)
- net ~INT2: now also U20B1.16 (~INT2)
- net ~INT3: now also U20B1.17 (~INT3)
- net ~INT6: now also U20B1.18 (~INT6)
- net ~IPL0: now also U20B1.13 (~IPL0)
- net ~IPL1: now also U20B1.14 (~IPL1)
- net ~IPL2: now also U20B1.15 (~IPL2)
- net ~LPEN: now also U19B1.37 (~LPEN)
- net ~RESET.P: now also U20B1.11 (~RESET)
- net ~VSYNC: now also U19B1.38 (~VSYNC)
- net ~ZD: now also U25B1.33 (~ZD)
- net +12V: now reaches J19.1 (Pin_1), R2.2
- net +BATT: no longer names the net of BT1.1 (+), BT1.2 (+), C30.1, R3.2
- net BATT+: no longer names the net of C23.1, CR1.1 (K), R3.1, U27.18 (VCC)
- net X2.C4 renamed C4b
- net X3.~RE renamed ~RE~b
- net X5.~RE renamed ~RE~c
- net X6.~CDW renamed ~CDW~b
- net X7.~CDW renamed ~CDW~c
- net X8.~CDW renamed ~CDW~d
- net X9.~CDW renamed ~CDW~e
Other:
- note removed: "SOCKET"
- moved on the sheet: R2
Changed lines of the file:
@@
 $EndDescr
 $Comp
-L Amiga-Rejuvenator:8361-Agnus U19B1
-U 1 1 5B8320A1
-P 23650 9500
-F 0 "U19B1" H 23650 10988 60  0000 C CNN
-F 1 "8361-Agnus" H 23200 11000 60  0001 L CNN
-F 2 "Package_DIP:DIP-48_W15.24mm_Socket" H 23000 8800 60  0001 C CNN
-F 3 "" H 23000 8800 60  0000 C CNN
-	1    23650 9500
-	1    0    0    -1
-$EndComp
-$Comp
 L Logic_Programmable:PAL16L8 U28
 U 1 1 5B83B1D0
@@
 Text Label 21675 9100 2    50   ~ 0
 D0
-$Comp
-L Amiga-Rejuvenator:8364-Paula U20B1
-U 1 1 5C2D1BFC
-P 18850 3900
-F 0 "U20B1" H 18850 5388 60  0000 C CNN
-F 1 "8364-Paula" H 18400 5400 60  0001 L CNN
-F 2 "MOLEX_4455:48pin_blank_socket" H 19500 3900 60  0001 C CNN
-F 3 "" H 19500 3900 60  0000 C CNN
-	1    18850 3900
-	1    0    0    -1
-$EndComp
-$Comp
-L Amiga-Rejuvenator:8362-Denise U25B1
-U 1 1 5C2D34C8
-P 18750 8900
-F 0 "U25B1" H 18750 10388 60  0000 C CNN
-F 1 "8362-Denise" H 18300 10400 60  0001 L CNN
-F 2 "MOLEX_4455:48pin_blank_socket" H 18100 8500 60  0001 C CNN
-F 3 "" H 18100 8500 60  0000 C CNN
-	1    18750 8900
-	1    0    0    -1
-$EndComp
 NoConn ~ 18200 3300
 NoConn ~ 18200 3400
@@
 Entry Wire Line
 	25150 17600 25250 17700
-Text Notes 18900 3375 1    118  ~ 0
-SOCKET
-Text Notes 18800 8300 1    118  ~ 0
-SOCKET
-Text Notes 23725 9125 1    118  ~ 0
-SOCKET
 $Comp
 L 74xx:74HC245 U34
@@
 PD15
 Text Label 6350 10450 2    50   ~ 0
-X8.~CDW
+~CDW~d
 Text Label 6350 10550 2    50   ~ 0
-X9.~CDW
+~CDW~e
 $Comp
 L power:+5V #PWR0206
@@
 XD6
 Text Label 6350 12250 2    50   ~ 0
-X6.~CDW
+~CDW~b
 Text Label 6350 12350 2    50   ~ 0
-X7.~CDW
+~CDW~c
 Text Label 6350 10250 2    50   ~ 0
 XD8
@@
 	10450 10450 9450 10450
 Text Label 4025 7850 0    50   ~ 0
-X2.C4
+C4b
 Text Label 4025 5850 0    50   ~ 0
-X5.~RE
+~RE~c
 Text Label 4025 7950 0    50   ~ 0
-X3.~RE
+~RE~b
 Entry Wire Line
 	5850 6550 5750 6650
@@
 L Device:R R2
 U 1 1 60DC1944
-P 7850 5000
-F 0 "R2" V 7750 4900 50  0000 L CNN
-F 1 "470" V 7850 4925 50  0000 L CNN
-F 2 "Resistor_THT:R_Axial_DIN0207_L6.3mm_D2.5mm_P15.24mm_Horizontal" V 7780 5000 50  0001 C CNN
-F 3 "~" H 7850 5000 50  0001 C CNN
-	1    7850 5000
+P 7900 5000
+F 0 "R2" V 7800 4900 50  0000 L CNN
+F 1 "470" V 7900 4900 50  0000 L CNN
+F 2 "Resistor_THT:R_Axial_DIN0207_L6.3mm_D2.5mm_P15.24mm_Horizontal" V 7830 5000 50  0001 C CNN
+F 3 "~" H 7900 5000 50  0001 C CNN
+	1    7900 5000
 	0    1    1    0
 $EndComp
@@
 P 7450 5000
 F 0 "J19" H 7500 4950 50  0001 R CNN
-F 1 "+12X" H 7500 5050 50  0000 R CNN
+F 1 "+12X" H 7450 5050 50  0000 R CNN
 F 2 "Connector_PinHeader_2.54mm:PinHeader_1x01_P2.54mm_Vertical" H 7450 5000 50  0001 C CNN
 F 3 "~" H 7450 5000 50  0001 C CNN
@@
 Wire Wire Line
 	24100 18500 25050 18500
-Wire Wire Line
-	7400 4200 7400 4250
-Wire Wire Line
-	7400 4250 7300 4250
 $Comp
 L Amiga-Rejuvenator:3.6V_Varta BT1
@@
 	-1   0    0    1
 $EndComp
-Wire Wire Line
-	7500 4200 7500 4250
-Wire Wire Line
-	7500 4250 7550 4250
-Wire Wire Line
-	7500 4250 7450 4250
-Connection ~ 7500 4250
-Connection ~ 7400 4250
 $Comp
 L Device:CP1_Small C39
@@
 Wire Wire Line
 	7900 4600 7900 4650
-Connection ~ 7900 4650
-Wire Wire Line
-	8050 4650 8050 5000
-Wire Wire Line
-	8050 5000 8000 5000
-Wire Wire Line
-	7900 4650 8050 4650
 Entry Wire Line
 	10450 6050 10550 5950
@@
 XD1
 Text Label 3100 12250 0    50   ~ 0
-X6.~CDW
+~CDW~b
 Text Label 3200 12850 0    50   ~ 0
 XD3
@@
 PD0
 Text Label 4350 12350 0    50   ~ 0
-X7.~CDW
+~CDW~c
 Wire Wire Line
 	2950 10050 3600 10050
@@
 $EndComp
 Text Label 3350 9350 0    50   ~ 0
-X8.~CDW
+~CDW~d
 Text Label 3400 9950 0    50   ~ 0
 XD12
@@
 PD15
 Text Label 4500 9450 0    50   ~ 0
-X9.~CDW
+~CDW~e
 $Comp
 L Amiga-Rejuvenator:Board2Board[20-pin] U38
@@
 RA7
 Text Label 2550 4850 0    50   ~ 0
-X5.~RE
+~RE~c
 Wire Wire Line
 	2550 7150 2900 7150
@@
 RA6
 Text Label 2550 6950 0    50   ~ 0
-X3.~RE
+~RE~b
 Wire Wire Line
 	1450 5250 1650 5250
@@
 A10
 Text Label 1650 6850 2    50   ~ 0
-X2.C4
+C4b
 Text Label 1550 6950 0    50   ~ 0
 A4
@@
 	-1   0    0    1
 $EndComp
-Connection ~ 7700 5000
+Wire Wire Line
+	7450 3750 7900 3750
 $Comp
-L power:PWR_FLAG #FLG0104
-U 1 1 61256223
-P 7450 4250
-F 0 "#FLG0104" H 7450 4325 50  0001 C CNN
-F 1 "PWR_FLAG" H 7200 4350 50  0000 C CNN
-F 2 "" H 7450 4250 50  0001 C CNN
-F 3 "~" H 7450 4250 50  0001 C CNN
-	1    7450 4250
-	-1   0    0    1
+L Amiga-Rejuvenator:8362-Denise-Socket U25B1
+U 1 1 63AA8453
+P 18750 8900
+F 0 "U25B1" H 18750 10388 60  0000 C CNN
+F 1 "8362-Denise-Socket" H 18300 10400 60  0001 L CNN
+F 2 "MOLEX_4455:48pin_blank_socket" H 18100 8500 60  0001 C CNN
+F 3 "" H 18100 8500 60  0000 C CNN
+	1    18750 8900
+	1    0    0    -1
+$EndComp
+$Comp
+L Amiga-Rejuvenator:8364-Paula-Socket U20B1
+U 1 1 63E982BC
+P 18850 3900
+F 0 "U20B1" H 18850 5388 60  0000 C CNN
+F 1 "8364-Paula-Socket" H 18400 5400 60  0001 L CNN
+F 2 "MOLEX_4455:48pin_blank_socket" H 19500 3900 60  0001 C CNN
+F 3 "" H 19500 3900 60  0000 C CNN
+	1    18850 3900
+	1    0    0    -1
 $EndComp
-Connection ~ 7450 4250
-Wire Wire Line
-	7450 4250 7400 4250
-Text Label 8250 4250 2    50   ~ 0
-BATT+
 $Comp
-L power:+BATT #PWR0129
-U 1 1 612661B9
-P 7300 4250
-F 0 "#PWR0129" H 7300 4100 50  0001 C CNN
-F 1 "+BATT" H 7300 4200 50  0000 C CNN
-F 2 "" H 7300 4250 50  0001 C CNN
-F 3 "" H 7300 4250 50  0001 C CNN
-	1    7300 4250
+L Amiga-Rejuvenator:8361-Agnus-Socket U19B1
+U 1 1 649700B7
+P 23650 9500
+F 0 "U19B1" H 23650 10988 60  0000 C CNN
+F 1 "8361-Agnus-Socket" H 23200 11000 60  0001 L CNN
+F 2 "Package_DIP:DIP-48_W15.24mm_Socket" H 25050 8800 60  0001 C CNN
+F 3 "" H 25050 8800 60  0000 C CNN
+	1    23650 9500
 	1    0    0    -1
 $EndComp
-Connection ~ 7300 4250
 Wire Wire Line
-	7300 4250 7200 4250
+	7200 4250 7400 4250
 Wire Wire Line
-	7450 3750 7900 3750
+	7400 4200 7400 4250
+Connection ~ 7400 4250
+Wire Wire Line
+	7400 4250 7500 4250
+Wire Wire Line
+	7500 4200 7500 4250
+Connection ~ 7500 4250
+Wire Wire Line
+	7500 4250 7550 4250
+Wire Wire Line
+	7700 5000 7750 5000
+Connection ~ 7700 5000
+Wire Wire Line
+	7900 4650 8100 4650
+Wire Wire Line
+	8100 4650 8100 5000
+Wire Wire Line
+	8100 5000 8050 5000
 Wire Wire Line
 	12400 13100 14350 13100
@@
 Wire Bus Line
 	13050 1250 13050 14200
+Connection ~ 7900 4650
+$Comp
+L power:+12V #PWR0129
+U 1 1 6786F0B6
+P 7700 5000
+F 0 "#PWR0129" H 7700 4850 50  0001 C CNN
+F 1 "+12V" H 7650 5150 50  0000 C CNN
+F 2 "" H 7700 5000 50  0001 C CNN
+F 3 "" H 7700 5000 50  0001 C CNN
+	1    7700 5000
+	1    0    0    -1
+$EndComp
 $EndSCHEMATC
