File: KiCAD/Amiga-Rejuvenator/Amiga-Rejuvenator.kicad_pcb (KiCad board)
At the start: 4 copper layers, 241.8 x 174.8 mm, 121 parts, among them J1 GND, J15 28M, J17 RMBCLKS, J18 GND, J19 +12X, U1 74LS245, U10 V53C104, U11 V53C104, U12 V53C104, U13 V53C104, U14 74LS244-U16,U17, U15 74LS373, U16 74LS244-U16,U17, U17 74LS244-U16,U17, U18 512K-ROM, U19 8372-FatAgnus, U19B1 8361-Agnus-Socket, U2 74LS393-U2, U20 8364-Paula, U20B1 8364-Paula-Socket, U21 74LS245, U22 74LS245, U23 RP, U24 RP, U25 8362-Denise, U25B1 8362-Denise-Socket, U26 74HC245, U27 OKI6242B, U28 PAL16L8, U29 PAL16L8, U3 74F257, U30 PAL20L8, U31 PAL20L8, U32 74LS74, U33 74LS04, U34 74HC245, U35 74F257, U36 PALCAS, U37 PALEN, U38 U3I, U39 U3G, U4 74LS244-U16,U17, U40 U2J, U41 U2I, U5 74LS373, U6 V53C104, U7 V53C104, U8 V53C104, U9 V53C104, X1 X1, X14 X14, X15 X15, X16 VideoSlot 1, X17 VideoSlot 2, Y1 Crystal

Commit message: Update board dimensions
Relocate post hole position slightly down and to the left.  Decrease width of upper right corner.   Increase width of bottom notch.

These locations had slight interference with the A1000 capacitors and posts, increasing the difficulty when installing Rejuvenator.   These dimensions have now been fine-tuned for better clearance.
Routing:
- net GND: vias 45 -> 44
Other:
- outline, holes or cut-outs redrawn
Changed lines of the file:
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@@
     (thickness 1.6)
     (drawings 136)
-    (tracks 3321)
+    (tracks 3320)
     (zones 0)
     (modules 121)
@@
       (net 6 +5V))
   )
+  (gr_line (start 304.038 53.848) (end 319.024 68.834) (layer Edge.Cuts) (width 0.15))
   (gr_text C1 (at 260.35 212.09) (layer F.SilkS)
     (effects (font (size 1 1) (thickness 0.15)))
@@
     (effects (font (size 1 1) (thickness 0.15)))
   )
-  (gr_line (start 305.435 53.848) (end 319.024 67.437) (layer Edge.Cuts) (width 0.15))
-  (gr_line (start 219.964 192.278) (end 219.964 227.838) (layer Edge.Cuts) (width 0.15))
-  (gr_line (start 209.804 227.838) (end 209.804 192.278) (layer Edge.Cuts) (width 0.15))
+  (gr_line (start 220.218 192.532) (end 220.218 227.838) (layer Edge.Cuts) (width 0.15))
+  (gr_line (start 209.296 227.838) (end 209.296 192.278) (layer Edge.Cuts) (width 0.15))
   (gr_text "EVERYTHING AMIGA!!!" (at 295.275 56.515) (layer F.SilkS)
     (effects (font (size 1 1) (thickness 0.25)))
@@
     (effects (font (size 1 1) (thickness 0.15)))
   )
-  (gr_text "JOETHEZOMBIE WAS HERE" (at 222.758 207.518 270) (layer F.Cu)
-    (effects (font (size 1.5 1.2) (thickness 0.25)))
+  (gr_text "JOETHEZOMBIE WAS HERE" (at 222.758 207.772 -90) (layer F.Cu)
+    (effects (font (size 1.7 1.2) (thickness 0.25)))
   )
   (gr_text RMBCLKS (at 236.22 211.328) (layer F.SilkS)
@@
   )
   (gr_line (start 318.135 228.6) (end 319.024 227.711) (layer Edge.Cuts) (width 0.15))
-  (gr_line (start 219.964 227.838) (end 220.726 228.6) (layer Edge.Cuts) (width 0.15))
-  (gr_line (start 219.456 191.77) (end 219.964 192.278) (layer Edge.Cuts) (width 0.15))
-  (gr_line (start 210.312 191.77) (end 219.456 191.77) (layer Edge.Cuts) (width 0.15))
-  (gr_line (start 209.042 228.6) (end 209.804 227.838) (layer Edge.Cuts) (width 0.15))
+  (gr_line (start 220.218 227.838) (end 220.98 228.6) (layer Edge.Cuts) (width 0.15))
+  (gr_line (start 219.456 191.77) (end 220.218 192.532) (layer Edge.Cuts) (width 0.15))
+  (gr_line (start 209.804 191.77) (end 219.456 191.77) (layer Edge.Cuts) (width 0.15))
+  (gr_line (start 208.534 228.6) (end 209.296 227.838) (layer Edge.Cuts) (width 0.15))
   (gr_line (start 77.216 227.965) (end 77.851 228.6) (layer Edge.Cuts) (width 0.15))
   (gr_line (start 77.851 174.879) (end 77.216 175.514) (layer Edge.Cuts) (width 0.15))
   (gr_line (start 114.3 173.99) (end 113.411 174.879) (layer Edge.Cuts) (width 0.15))
   (gr_line (start 116.84 53.975) (end 114.3 56.515) (layer Edge.Cuts) (width 0.15))
-  (gr_circle (center 175.387 184.261117) (end 180.848 187.325) (layer Edge.Cuts) (width 0.15))
+  (gr_circle (center 175.09422 184.658) (end 180.55522 187.721883) (layer Edge.Cuts) (width 0.15))
   (gr_line (start 77.216 175.514) (end 77.216 227.965) (layer Edge.Cuts) (width 0.15))
   (gr_line (start 113.411 174.879) (end 77.851 174.879) (layer Edge.Cuts) (width 0.15))
   (gr_line (start 114.3 56.515) (end 114.3 173.99) (layer Edge.Cuts) (width 0.15))
-  (gr_line (start 305.435 53.848) (end 116.84 53.975) (layer Edge.Cuts) (width 0.15))
-  (gr_line (start 319.024 227.711) (end 319.024 67.437) (layer Edge.Cuts) (width 0.15))
-  (gr_line (start 220.726 228.6) (end 318.135 228.6) (layer Edge.Cuts) (width 0.15))
-  (gr_line (start 209.804 192.278) (end 210.312 191.77) (layer Edge.Cuts) (width 0.15))
-  (gr_line (start 77.851 228.6) (end 209.042 228.6) (layer Edge.Cuts) (width 0.15))
+  (gr_line (start 304.038 53.848) (end 116.84 53.975) (layer Edge.Cuts) (width 0.15))
+  (gr_line (start 319.024 227.711) (end 319.024 68.834) (layer Edge.Cuts) (width 0.15))
+  (gr_line (start 220.98 228.6) (end 318.135 228.6) (layer Edge.Cuts) (width 0.15))
+  (gr_line (start 209.296 192.278) (end 209.804 191.77) (layer Edge.Cuts) (width 0.15))
+  (gr_line (start 77.851 228.6) (end 208.534 228.6) (layer Edge.Cuts) (width 0.15))
   (segment (start 255.27 209.55) (end 250.19 204.47) (width 0.25) (layer F.Cu) (net 1) (status 30))
   (segment (start 255.27 212.09) (end 255.27 209.55) (width 1.5) (layer In2.Cu) (net 1) (status 30))
@@
   (via (at 205.74 217.17) (size 0.8) (drill 0.4) (layers F.Cu B.Cu) (net 2))
   (via (at 207.01 217.17) (size 0.8) (drill 0.4) (layers F.Cu B.Cu) (net 2))
-  (via (at 208.28 217.17) (size 0.8) (drill 0.4) (layers F.Cu B.Cu) (net 2))
   (via (at 204.47 218.44) (size 0.8) (drill 0.4) (layers F.Cu B.Cu) (net 2))
   (via (at 203.2 218.44) (size 0.8) (drill 0.4) (layers F.Cu B.Cu) (net 2))
@@
   )
   (zone (net 2) (net_name GND) (layer In1.Cu) (hatch edge 0.508)
-    (connect_pads thru_hole_only (clearance 0.34))
-    (min_thickness 0.254)
-    (fill yes (arc_segments 16) (thermal_gap 0.5) (thermal_bridge_width 0.508) (smoothing chamfer) (radius 0.1))
-    (polygon
-      (pts
-        (xy 204.47 94.488) (xy 204.216 94.742) (xy 204.216 96.139) (xy 204.216 97.79) (xy 204.216 98.552)
-        (xy 204.216 132.334) (xy 201.676 135.128) (xy 201.676 184.15) (xy 201.168 184.658) (xy 201.168 191.77)
-        (xy 200.533 192.532) (xy 197.231 192.532) (xy 194.945 195.326) (xy 194.945 224.155) (xy 195.58 224.79)
-        (xy 198.628 224.79) (xy 199.39 224.155) (xy 199.39 220.98) (xy 200.66 219.71) (xy 203.2 219.71)
-        (xy 204.47 220.98) (xy 204.47 227.33) (xy 208.28 227.33) (xy 208.28 218.694) (xy 209.042 218.186)
-        (xy 209.042 216.662) (xy 208.788 216.408) (xy 200.66 216.408) (xy 198.882 214.884) (xy 199.136 199.39)
-        (xy 202.438 195.58) (xy 204.978 195.58) (xy 209.55 190.5) (xy 219.456 190.5) (xy 220.218 191.262)
-        (xy 220.218 225.298) (xy 220.98 226.06) (xy 224.79 226.06) (xy 225.298 225.552) (xy 225.298 182.88)
-        (xy 224.028 181.61) (xy 208.026 181.61) (xy 206.248 179.832) (xy 206.248 135.128) (xy 209.042 132.588)
-        (xy 209.042 94.996) (xy 208.534 94.488)
-      )
-    )
-  )
-  (zone (net 2) (net_name GND) (layer In1.Cu) (hatch edge 0.508)
     (connect_pads thru_hole_only (clearance 0.5))
     (min_thickness 0.254)
@@
     (polygon
       (pts
-        (xy 314.198 64.77) (xy 314.198 90.17) (xy 317.5 92.71) (xy 317.5 96.012) (xy 312.42 101.092)
+        (xy 314.198 65.024) (xy 314.198 90.17) (xy 317.5 92.71) (xy 317.5 96.012) (xy 312.42 101.092)
         (xy 312.42 109.22) (xy 313.69 110.49) (xy 314.96 110.49) (xy 318.77 114.3) (xy 318.77 121.92)
         (xy 316.992 123.698) (xy 308.356 123.698) (xy 306.832 125.222) (xy 306.832 141.478) (xy 304.8 143.51)
@@
     (polygon
       (pts
-        (xy 304.8 54.356) (xy 309.372 58.928) (xy 309.372 67.056) (xy 307.34 69.088) (xy 304.546 66.04)
+        (xy 303.53 54.356) (xy 309.372 60.198) (xy 309.372 67.056) (xy 307.34 69.088) (xy 304.546 66.04)
         (xy 297.688 66.04) (xy 294.64 69.088) (xy 291.592 66.04) (xy 284.988 66.04) (xy 281.94 69.088)
         (xy 278.892 66.04) (xy 272.288 66.04) (xy 269.24 69.088) (xy 266.192 66.04) (xy 259.588 66.04)
@@
         (xy 248.412 194.31) (xy 247.142 193.04) (xy 239.268 193.04) (xy 237.49 194.818) (xy 234.95 194.818)
         (xy 233.172 193.04) (xy 232.918 193.04) (xy 231.14 194.818) (xy 228.6 194.818) (xy 226.822 193.04)
-        (xy 221.234 193.04) (xy 219.456 191.516) (xy 210.312 191.516) (xy 208.788 193.04) (xy 208.788 197.866)
+        (xy 221.488 193.04) (xy 219.71 191.262) (xy 209.804 191.262) (xy 208.788 192.278) (xy 208.788 197.866)
         (xy 208.026 198.628) (xy 205.994 198.628) (xy 205.232 197.866) (xy 205.232 195.58) (xy 204.216 194.818)
         (xy 202.184 194.818) (xy 201.168 195.58) (xy 201.168 197.612) (xy 199.39 199.39) (xy 181.864 199.39)
@@
         (xy 90.17 199.898) (xy 87.63 199.898) (xy 87.122 199.39) (xy 87.122 196.85) (xy 90.932 193.04)
         (xy 115.57 193.04) (xy 116.84 191.77) (xy 142.24 191.77) (xy 143.256 190.754) (xy 165.1 190.754)
-        (xy 167.64 189.23) (xy 170.18 190.754) (xy 185.166 190.754) (xy 186.69 192.278) (xy 205.232 192.278)
+        (xy 167.64 189.23) (xy 170.942 191.262) (xy 185.166 191.262) (xy 186.182 192.278) (xy 205.232 192.278)
         (xy 205.994 191.516) (xy 205.994 180.34) (xy 254 180.34) (xy 257.81 184.15) (xy 274.32 184.15)
         (xy 276.098 182.372)
@@
       )
     )
+  )
+  (zone (net 2) (net_name GND) (layer In1.Cu) (hatch edge 0.508)
+    (connect_pads thru_hole_only (clearance 0.34))
+    (min_thickness 0.254)
+    (fill yes (arc_segments 16) (thermal_gap 0.5) (thermal_bridge_width 0.508) (smoothing chamfer) (radius 0.1))
+    (polygon
+      (pts
+        (xy 204.47 94.488) (xy 204.216 94.742) (xy 204.216 96.139) (xy 204.216 97.79) (xy 204.216 98.552)
+        (xy 204.216 132.334) (xy 201.676 135.128) (xy 201.676 184.15) (xy 201.168 184.658) (xy 201.168 191.77)
+        (xy 200.533 192.532) (xy 197.231 192.532) (xy 194.945 195.326) (xy 194.945 224.155) (xy 195.58 224.79)
+        (xy 198.628 224.79) (xy 199.39 224.155) (xy 199.39 220.98) (xy 200.66 219.71) (xy 203.2 219.71)
+        (xy 204.47 220.98) (xy 204.47 227.33) (xy 208.28 227.33) (xy 208.28 218.694) (xy 208.28 218.186)
+        (xy 208.28 216.916) (xy 207.772 216.408) (xy 200.66 216.408) (xy 198.882 214.884) (xy 199.136 199.39)
+        (xy 202.438 195.58) (xy 204.978 195.58) (xy 209.55 190.5) (xy 219.456 190.5) (xy 220.472 191.516)
+        (xy 220.472 225.552) (xy 220.98 226.06) (xy 224.79 226.06) (xy 225.298 225.552) (xy 225.298 182.88)
+        (xy 224.028 181.61) (xy 208.026 181.61) (xy 206.248 179.832) (xy 206.248 135.128) (xy 209.042 132.588)
+        (xy 209.042 94.996) (xy 208.534 94.488)
+      )
+    )

Commit message: Update board artwork
Other:
- board text added: "PLD Zone demystified by scrollreader Matthias"

Commit message: Update board artwork
Other:
- board text added: "01100111 01110010 01100101 01100111 01110100 01101001 01100010 01100010 01110011 00101000 00110001 00111001 00110101 00111001 00101101 00110010 00110000 00110010 00110000 00101001"
- board text added: "Greg Tibbs (1959-2020)"
- board text added: "Matthias Heinrichs Christian Stich Matt Martin Marco Both Adrian Garay & Eric Hill"
- board text added: "Project Support By:"
